File: Motor_Control/Motor_Control.kicad_pcb (KiCad board)
At the start: 2 copper layers, 56 x 129.5 mm, 33 parts, among them J1 Conn_01x06_Male, J2 Conn_01x06_Male, J3 Conn_01x06_Male, J4 Conn_01x04_Male, J5 Conn_01x03_Female, J6 Conn_02x05_Odd_Even, J7 Conn_02x05_Odd_Even, J8 Screw_Terminal_01x02, Q1 BSS138, Q2 BSS138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

Commit message: Update layout files
Routing:
- net /SERVO: track 40.2 -> 41.2 mm
- net /STEP: track 59.9 -> 60.9 mm
- net /STEP_DIR: track 64.8 -> 65.7 mm
Other:
- board text added: "03/15/19"
- board text added: "Benjamin Ward"
- board text added: "M1"
- board text added: "M2"
- board text added: "M3"
- board text added: "Motor Control Breakout Rev 2"
- board text added: "SS"
- board text added: "WPI RBE 2002 D19"
- board text added: "https://github.com/WardBenjamin/RBE2002_SpiderwebPCB"
