File: Spiderweb_RIB_Shield/Spiderweb.kicad_pcb (KiCad board)
At the start: 2 copper layers, 66 x 50.8 mm, 14 parts, among them J1 Conn_02x05_Odd_Even, J10 Conn_01x04_Female, J2 Conn_02x05_Odd_Even, J3 Conn_01x19_Female, J4 Conn_01x19_Female, J5 Conn_01x19_Female, J6 Conn_01x19_Female, J7 Conn_01x19_Female, J8 Conn_01x19_Female, J9 Conn_01x04_Female

Commit message: Update layout files
Other:
- board text added: "03/15/19"
- board text added: "Benjamin Ward"
- board text added: "Spiderweb Shield Rev 3"
- board text added: "WPI RBE 2002 D19"
- board text added: "https://github.com/WardBenjamin/RBE2002_SpiderwebPCB"
Changed lines of the file:
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@@
   (general
     (thickness 1.6)
-    (drawings 4)
+    (drawings 9)
     (tracks 238)
     (zones 0)
@@
     )
   )
+  (gr_text 03/15/19 (at 150.823326 92.88663) (layer F.SilkS)
+    (effects (font (size 1.5 1.5) (thickness 0.3)))
+  )
+  (gr_text "WPI RBE 2002 D19" (at 147.648326 89.33063) (layer F.SilkS)
+    (effects (font (size 1.25 1.25) (thickness 0.25)))
+  )
+  (gr_text "Spiderweb Shield Rev 3" (at 120.851326 89.33063) (layer F.SilkS)
+    (effects (font (size 1.25 1.25) (thickness 0.3)))
+  )
+  (gr_text https://github.com/WardBenjamin/RBE2002_SpiderwebPCB (at 117.549326 90.72763) (layer F.SilkS)
+    (effects (font (size 0.35 0.35) (thickness 0.0875)))
+  )
+  (gr_text "Benjamin Ward" (at 117.803326 92.88663) (layer F.SilkS)
+    (effects (font (size 1.5 1.5) (thickness 0.3)))
+  )
   (gr_line (start 100.023326 43.99163) (end 166.063326 43.99163) (layer Edge.Cuts) (width 0.15))
